File: elec/layout/default/tps63020dsjr.kicad_pcb (KiCad board)
At the start: 2 copper layers, 225.7 x 100.8 mm, 10 parts

Commit message: Remove crud from layout
Other:
- board outline removed
- board text removed: "{{GITHASH}}"
